File: hw/Breakout.kicad_pcb (KiCad board)
At the start: 2 copper layers, 34.2 x 34.4 mm, 22 parts, among them IC1 AP2112K-3.3TRG1, J1 ST60X-18S30, J2 SJ-3523-SMT-TR, J3 BM03B-SRSS-TBT_LF__SN_, J4 BM03B-SRSS-TBT_LF__SN_, J5 SJ-3523-SMT-TR, J6 SM04B-SRSS-TB_LF__SN_, U1 12401610E4-2A, U2 74LVC1G00, U3 74LVC1G06

Commit message: revised design
Parts:
- moved S2 3.93 mm to (107.7, 96.9)
- moved J1 2.99 mm to (97.0, 100.0)
- moved FB1 2.78 mm to (109.4, 89.6)
- moved FB2 2.78 mm to (113.8, 89.6)
- moved R3 2.78 mm to (111.0, 89.0)
- moved R4 2.78 mm to (112.1, 89.0)
Connections:
- net I2C0_SDL renamed I2C0_SCL
- J2 pad 2: /HP_L -> /HP_R
- J2 pad 3: /HP_R -> /HP_L
Routing:
- net /HP_R: track 30.2 -> 17.5 mm
- net UART0_RX: track 15.3 -> 27.4 mm, vias 2 -> 0
- net I2C0_SDA: track 16.5 -> 10.7 mm, vias 2 -> 0
- net I2C0_SCL: track 14.9 -> 9.71 mm, vias 2 -> 0
- net UART1_TX: track 19.5 -> 24.6 mm, vias 0 -> 2
- net J5_TIP: track 14.5 -> 9.97 mm
- net UART0_TX: track 15.8 -> 20.2 mm, vias 2 -> 0
- net SWD: track 12.8 -> 17.1 mm
- net IN2_L: track 20.4 -> 24.7 mm
- net IN2_R: track 17.9 -> 21.2 mm
- net SWCLK: track 16.7 -> 14.1 mm
- net /BOOTSEL: track 10.3 -> 12.9 mm, vias 2 -> 3
- net USB_D+: track 32.9 -> 31.2 mm
- net /HP_L: track 25.7 -> 27.3 mm
- net MIDI_TX: track 6.16 -> 4.58 mm
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Other:
- board size 34.2 x 34.4 mm -> 34.2 x 33.4 mm
- board text added: "AUDIO ↓↑ MIDI"
- board text added: "I2C0"
- board text added: "PicoPCMCIA Breakout v1.1"
- board text added: "SWD"
- board text added: "UART0"
- board text removed: "AUDIO IN↓↑MIDI OUT"
- board text removed: "PicoPCMCIA Breakout v1"
