File: hw/Breakout.kicad_pcb (KiCad board)
At the start: 2 copper layers, 34.2 x 33.4 mm, 22 parts, among them IC1 AP2112K-3.3TRG1, J1 ST60X-18S30, J2 SJ-3523-SMT-TR, J3 BM03B-SRSS-TBT_LF__SN_, J4 BM03B-SRSS-TBT_LF__SN_, J5 SJ-3523-SMT-TR, J6 SM04B-SRSS-TB_LF__SN_, U1 12401610E4-2A, U2 74LVC1G00, U3 74LVC1G06

Commit message: hw: J2/J5 -> SJ-3524-SMT-TR (C20182907, in stock); routing to follow
SJ-3523-SMT-TR (C4991872) has no JLC stock.  The SJ-3524 is the same
Same Sky SJ-352X-SMT body with a tip-switch terminal, pin 4, behind the
jack: footprint BreakoutLibrary:SJ3524SMTTR, pad 4 left unconnected.

Not routed yet.  Pad 4 sits on J6 pad 1 and the +3.3V/GND tracks and via
behind J2, and on R3/R4/FB2 and their tracks and via behind J5: 43 new DRC
items, all on pad 4.

Co-Authored-By: Claude Opus 5.5 <noreply@anthropic.com>
Claude-Session: https://claude.ai/code/session_0133r6nzUahChJ5bbJy715cX
Parts:
- J2, J5: value SJ-3523-SMT-TR -> SJ-3524-SMT-TR; footprint BreakoutLibrary:SJ3523SMTTR -> BreakoutLibrary:SJ3524SMTTR
Changed lines of the file:
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@@
 	(net 40 "/HP_L")
 	(net 41 "unconnected-(J1-Pad12)")
-	(footprint "BreakoutLibrary:SJ3523SMTTR"
+	(footprint "BreakoutLibrary:SJ3524SMTTR"
 		(layer "F.Cu")
 		(at 111.225 72.5 -90)
-		(descr "SJ-3523-SMT-TR-1")
+		(descr "SJ-3524-SMT-TR")
 		(tags "Connector")
 		(property "Reference" "J5"
@@
 			)
 		)
-		(property "Value" "SJ-3523-SMT-TR"
+		(property "Value" "SJ-3524-SMT-TR"
 			(at 7.3 0.4 90)
 			(layer "F.SilkS")
@@
 			)
 		)
-		(property "Datasheet" "https://www.sameskydevices.com/product/resource/SJ-3523-SMT-TR.pdf"
+		(property "Datasheet" "https://www.sameskydevices.com/product/resource/sj-352x-smt.pdf"
 			(at 0 0 90)
 			(layer "F.Fab")
@@
 			)
 		)
-		(property "Description" "SJ-3523-SMT-TR - 3.5 mm, Stereo, Right Angle, Surface Mount (SMT), 3 Conductors, 0 Internal Switches, Audio Jack Connector"
+		(property "Description" "SJ-3524-SMT-TR - 3.5 mm, Stereo, Right Angle, Surface Mount (SMT), 3 Conductors, 1 Internal Switch (tip), Audio Jack Connector"
 			(at 0 0 90)
 			(layer "F.Fab")
@@
 			)
 		)
-		(property "Mouser Part Number" "490-SJ-3523-SMT-TR"
+		(property "Mouser Part Number" "490-SJ-3524-SMT-TR"
 			(at 0 0 270)
 			(unlocked yes)
@@
 			)
 		)
-		(property "Mouser Price/Stock" "https://www.mouser.co.uk/ProductDetail/CUI-Devices/SJ-3523-SMT-TR?qs=WyjlAZoYn51zOHzJ3r4ZRA%3D%3D"
+		(property "Mouser Price/Stock" "https://www.mouser.com/ProductDetail/Same-Sky/SJ-3524-SMT-TR"
 			(at 0 0 270)
 			(unlocked yes)
@@
 			)
 		)
-		(property "Manufacturer_Part_Number" "SJ-3523-SMT-TR"
+		(property "Manufacturer_Part_Number" "SJ-3524-SMT-TR"
 			(at 0 0 270)
 			(unlocked yes)
@@
 		(sheetname "/")
 		(sheetfile "Breakout.kicad_sch")
-		(property "LCSC" "C4991872"
+		(property "LCSC" "C20182907"
 			(at 0 0 0)
 			(layer "F.Fab")
@@
 		(fp_line
 			(start 14.5 3.05)
-			(end 14.5 1.5)
+			(end 14.5 0.9)
 			(stroke
 				(width 0.1)
@@
 		(fp_line
 			(start 14.5 -3)
-			(end 14.5 1.5)
+			(end 14.5 -2.4)
 			(stroke
 				(width 0.1)
@@
 			(pintype "passive")
 		)
+		(pad "4" smd rect
+			(at 15.8 -0.75 270)
+			(size 2.6 2.8)
+			(layers "F.Cu" "F.Mask" "F.Paste")
+		)
 		(embedded_fonts no)
 		(model "SJ-3523-SMT-TR.stp"
@@
 		)
 	)
-	(footprint "BreakoutLibrary:SJ3523SMTTR"
+	(footprint "BreakoutLibrary:SJ3524SMTTR"
 		(layer "F.Cu")
 		(at 88.525 72.5 -90)
-		(descr "SJ-3523-SMT-TR-1")
+		(descr "SJ-3524-SMT-TR")
 		(tags "Connector")
 		(property "Reference" "J2"
@@
 			)
 		)
-		(property "Value" "SJ-3523-SMT-TR"
+		(property "Value" "SJ-3524-SMT-TR"
 			(at 7.3 0.4 90)
 			(layer "F.SilkS")
@@
 			)
 		)
-		(property "Datasheet" "https://www.sameskydevices.com/product/resource/SJ-3523-SMT-TR.pdf"
+		(property "Datasheet" "https://www.sameskydevices.com/product/resource/sj-352x-smt.pdf"
 			(at 0 0 90)
 			(layer "F.Fab")
@@
 			)
 		)
-		(property "Description" "SJ-3523-SMT-TR - 3.5 mm, Stereo, Right Angle, Surface Mount (SMT), 3 Conductors, 0 Internal Switches, Audio Jack Connector"
+		(property "Description" "SJ-3524-SMT-TR - 3.5 mm, Stereo, Right Angle, Surface Mount (SMT), 3 Conductors, 1 Internal Switch (tip), Audio Jack Connector"
 			(at 0 0 90)
 			(layer "F.Fab")
@@
 			)
 		)
-		(property "Mouser Part Number" "490-SJ-3523-SMT-TR"
+		(property "Mouser Part Number" "490-SJ-3524-SMT-TR"
 			(at 0 0 270)
 			(unlocked yes)
@@
 			)
 		)
-		(property "Mouser Price/Stock" "https://www.mouser.co.uk/ProductDetail/CUI-Devices/SJ-3523-SMT-TR?qs=WyjlAZoYn51zOHzJ3r4ZRA%3D%3D"
+		(property "Mouser Price/Stock" "https://www.mouser.com/ProductDetail/Same-Sky/SJ-3524-SMT-TR"
 			(at 0 0 270)
 			(unlocked yes)
@@
 			)
 		)
-		(property "Manufacturer_Part_Number" "SJ-3523-SMT-TR"
+		(property "Manufacturer_Part_Number" "SJ-3524-SMT-TR"
 			(at 0 0 270)
 			(unlocked yes)
@@
 		(sheetname "/")
 		(sheetfile "Breakout.kicad_sch")
-		(property "LCSC" "C4991872"
+		(property "LCSC" "C20182907"
 			(at 0 0 0)
 			(layer "F.Fab")
@@
 		(fp_line
 			(start 14.5 3.05)
-			(end 14.5 1.5)
+			(end 14.5 0.9)
 			(stroke
 				(width 0.1)
@@
 		(fp_line
 			(start 14.5 -3)
-			(end 14.5 1.5)
+			(end 14.5 -2.4)
 			(stroke
 				(width 0.1)
@@
 			(pintype "passive")
 		)
+		(pad "4" smd rect
+			(at 15.8 -0.75 270)
+			(size 2.6 2.8)
+			(layers "F.Cu" "F.Mask" "F.Paste")
+		)
 		(embedded_fonts no)
