File: hw/Breakout.kicad_sch (KiCad schematic)
At the start: 7 parts, among them J1 ST60X-18S30, J2 SJ-3523-SMT-TR, J3 BM03B-SRSS-TBT_LF__SN_, U1 12401610E4-2A

Commit message: Work in progress
Parts:
- added C1, C2, C5: 0.1uF, Capacitor_SMD:C_0402_1005Metric, symbol Device:C
- added C3: 1uF, Capacitor_SMD:C_0402_1005Metric, symbol Device:C
- added FB1, FB2: 1KΩ@100MHz, Inductor_SMD:L_0805_2012Metric, symbol Device:FerriteBead
- added IC1: AP2112K-3.3TRG1, BreakoutLibrary:SOT95P285X140-5N, symbol BreakoutLibrary:AP2112K-3.3TRG1
- added J4: BM03B-SRSS-TBT_LF__SN_, BreakoutLibrary:BM03BSRSSTBTLFSN, symbol DongleLibrary:BM03B-SRSS-TBT_LF__SN_
- added J5: SJ-3523-SMT-TR, BreakoutLibrary:SJ3523SMTTR, symbol DongleLibrary:SJ-3523-SMT-TR
- added J6: SM04B-SRSS-TB_LF__SN_, BreakoutLibrary:SM04B-SRSS-TB_LFSN_, symbol BreakoutLibrary:SM04B-SRSS-TB_LF__SN_
- added R3, R4: 220, Resistor_SMD:R_0402_1005Metric, symbol Device:R
- added S2: JS202011SCQN, BreakoutLibrary:JS202011SCQN, symbol BreakoutLibrary:JS202011SCQN
- added U2: 74LVC1G00, Package_TO_SOT_SMD:SOT-353_SC-70-5, symbol 74xGxx:74LVC1G00
- added U3: 74LVC1G06, Package_TO_SOT_SMD:TSOT-23-5, symbol 74xGxx:74LVC1G06
Connections:
- net SWDIO is gone; now on net SWD: J1.2
- net GND: now also J3.2, J3.4 (MP1), J3.5 (MP2), C1.2, C2.2, C3.2, C5.2, IC1.2 (GND), J4.2, J4.4 (MP1), J4.5 (MP2), J5.1 (SLEEVE), J6.1, U2.3 (GND), U3.3 (GND)
- net HP_L: now also J1.16, J2.2 (TIP)
- net HP_R: now also J1.17, J2.3 (RING)
- net I2C0_SDA: now also J6.3
- net I2C0_SDL: now also J6.4
- net IN2_L: now also J1.14, S2.3
- net IN2_R: now also J1.15, S2.6
- net SWCLK: now also J3.1
- net UART0_RX: now also J4.1
- net UART0_TX: now also J4.3
- net UART1_TX: now also U2.1, U2.2
- net SWD: now reaches J3.3
- net USB_VBUS renamed +5V
- net +5V: now also C1.1, C2.1, C5.1, IC1.1 (VIN), IC1.3 (EN), R4.2, U2.5 (VCC), U3.5 (VCC)
- new net: U2.4, U3.2
- new net: R3.1, U3.4
- new net: FB1.1, R3.2
- new net: FB2.1, R4.1
- new net +3.3V: C3.1, IC1.5 (VOUT), J6.2
- new net J5_RING: J5.3 (RING), S2.5
- new net J5_TIP: J5.2 (TIP), S2.2
- new net MIDI_5V: FB2.2, S2.4
- new net MIDI_TX: FB1.2, S2.1
Other:
- note added: "MIDI/DEBUG OUT"
- moved on the sheet: J3
