File: hw/Breakout.kicad_sch (KiCad schematic)
At the start: 22 parts, among them IC1 AP2112K-3.3TRG1, J1 ST60X-18S30, J2 SJ-3523-SMT-TR, J3 BM03B-SRSS-TBT_LF__SN_, J4 BM03B-SRSS-TBT_LF__SN_, J5 SJ-3523-SMT-TR, J6 SM04B-SRSS-TB_LF__SN_, U1 12401610E4-2A, U2 74LVC1G00, U3 74LVC1G06

Commit message: revised design
Connections:
- net HP_L: now also J2.3 (RING); no longer J2.2 (TIP)
- net HP_R: now also J2.2 (TIP); no longer J2.3 (RING)
- net I2C0_SDL renamed I2C0_SCL
Other:
- moved on the sheet: J2
