File: hw/Breakout.kicad_sch (KiCad schematic)
At the start: 22 parts, among them IC1 AP2112K-3.3TRG1, J1 ST60X-18S30, J2 SJ-3523-SMT-TR, J3 BM03B-SRSS-TBT_LF__SN_, J4 BM03B-SRSS-TBT_LF__SN_, J5 SJ-3523-SMT-TR, J6 SM04B-SRSS-TB_LF__SN_, U1 12401610E4-2A, U2 74LVC1G00, U3 74LVC1G06

Commit message: hw: LCSC numbers fixed for JLC stock (breakout)
Out of stock / wrong part:
- U2  74LVC1G00: C2878883 (DCKT, 1 in stock) -> C8185 SN74LVC1G00DCKR
- IC1 AP2112K-3.3TRG1: C23380830 (TECH PUBLIC clone) -> C51118 (Diodes,
  the part already held in the JLC private stock)
- J1  ST60X-18S(30): had no LCSC -> C21136285 (held in private stock)
- FB1/FB2 1k@100MHz: C16903 was BLM21PG300 (30 ohm) -> C85835 BLM21AG102SN1D
- R3/R4 220: C114764 was 200 ohm -> C25091 (220 ohm, basic)

Extended -> basic:
- C1/C2/C5 0.1uF 0402 -> C1525; C3 1uF 0402 -> C52923; R1/R2 5.1K -> C25905

J2/J5 keep SJ-3523-SMT-TR (C4991872, 0 at JLC: global sourcing).  LCSC is
now also on the board and in the schematic for every placed part.

BreakoutLibrary: SJ3524SMTTR footprint (SJ-3523 + tip-switch pad 4 at
15.8,-0.75 from the EasyEDA land pattern), not used yet: its pad 4 lands
on R3/R4/FB2/J6 in the current layout.

DRC (with schematic parity) and ERC counts unchanged.

Co-Authored-By: Claude Opus 5.5 <noreply@anthropic.com>
Claude-Session: https://claude.ai/code/session_0133r6nzUahChJ5bbJy715cX
Parts:
- C1, C2, C5: LCSC (none) -> C1525
- C3: LCSC (none) -> C52923
- FB1, FB2: LCSC (none) -> C85835
- IC1: LCSC (none) -> C51118
- J1: LCSC (none) -> C21136285
- J2, J5: LCSC (none) -> C4991872
- J3, J4: LCSC (none) -> C495538
- J6: LCSC (none) -> C160404
- R1, R2: LCSC (none) -> C25905
- R3, R4: LCSC (none) -> C25091
- S1: LCSC (none) -> C139797
- S2: LCSC (none) -> C221666
- U1: LCSC (none) -> C5119948
- U2: LCSC (none) -> C8185
- U3: LCSC (none) -> C840103
Changed lines of the file:
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@@
+			)
+		)
+		(property "LCSC" "C8185"
+			(at 68.58 172.72 0)
+			(effects
+				(font
+					(size 1.27 1.27)
+				)
+				(hide yes)
 			)
 		)
@@
 			)
 		)
+		(property "LCSC" "C4991872"
+			(at 73.66 68.58 0)
+			(effects
+				(font
+					(size 1.27 1.27)
+				)
+				(hide yes)
+			)
+		)
 		(pin "1"
 		)
@@
 			)
 		)
+		(property "LCSC" "C4991872"
+			(at 217.17 154.94 0)
+			(effects
+				(font
+					(size 1.27 1.27)
+				)
+				(hide yes)
+			)
+		)
 		(pin "1"
 		)
@@
 			)
 		)
+		(property "LCSC" "C1525"
+			(at 55.88 154.94 0)
+			(effects
+				(font
+					(size 1.27 1.27)
+				)
+				(hide yes)
+			)
+		)
 		(pin "1"
 		)
@@
 		)
 		(property "Description" ""
+			(at 36.83 109.22 0)
+			(effects
+				(font
+					(size 1.27 1.27)
+				)
+				(hide yes)
+			)
+		)
+		(property "LCSC" "C21136285"
 			(at 36.83 109.22 0)
 			(effects
@@
 			)
 		)
+		(property "LCSC" "C495538"
+			(at 133.35 48.26 0)
+			(effects
+				(font
+					(size 1.27 1.27)
+				)
+				(hide yes)
+			)
+		)
 		(pin "3"
 		)
@@
 			)
 		)
+		(property "LCSC" "C52923"
+			(at 180.34 116.84 0)
+			(effects
+				(font
+					(size 1.27 1.27)
+				)
+				(hide yes)
+			)
+		)
 		(pin "1"
 		)
@@
 			)
 		)
+		(property "LCSC" "C495538"
+			(at 133.35 24.13 0)
+			(effects
+				(font
+					(size 1.27 1.27)
+				)
+				(hide yes)
+			)
+		)
 		(pin "3"
 		)
@@
 			)
 		)
+		(property "LCSC" "C5119948"
+			(at 226.06 30.48 0)
+			(effects
+				(font
+					(size 1.27 1.27)
+				)
+				(hide yes)
+			)
+		)
 		(pin "A2"
 		)
@@
 			)
 		)
+		(property "LCSC" "C25091"
+			(at 118.11 172.72 0)
+			(effects
+				(font
+					(size 1.27 1.27)
+				)
+				(hide yes)
+			)
+		)
 		(pin "1"
 		)
@@
 			)
 		)
+		(property "LCSC" "C25091"
+			(at 123.19 156.21 0)
+			(effects
+				(font
+					(size 1.27 1.27)
+				)
+				(hide yes)
+			)
+		)
 		(pin "1"
 		)
@@
 			)
 		)
+		(property "LCSC" "C25905"
+			(at 205.74 40.64 0)
+			(effects
+				(font
+					(size 1.27 1.27)
+				)
+				(hide yes)
+			)
+		)
 		(pin "2"
 		)
@@
 			)
 		)
+		(property "LCSC" "C160404"
+			(at 135.89 76.2 0)
+			(effects
+				(font
+					(size 1.27 1.27)
+				)
+				(hide yes)
+			)
+		)
 		(pin "4"
 		)
@@
 			)
 		)
+		(property "LCSC" "C51118"
+			(at 142.24 106.68 0)
+			(effects
+				(font
+					(size 1.27 1.27)
+				)
+				(hide yes)
+			)
+		)
 		(pin "1"
 		)
@@
 			)
 		)
+		(property "LCSC" "C1525"
+			(at 128.27 115.57 0)
+			(effects
+				(font
+					(size 1.27 1.27)
+				)
+				(hide yes)
+			)
+		)
 		(pin "1"
 		)
@@
 			)
 		)
+		(property "LCSC" "C1525"
+			(at 48.26 154.94 0)
+			(effects
+				(font
+					(size 1.27 1.27)
+				)
+				(hide yes)
+			)
+		)
 		(pin "1"
 		)
@@
 			)
 		)
+		(property "LCSC" "C85835"
+			(at 128.27 172.72 0)
+			(effects
+				(font
+					(size 1.27 1.27)
+				)
+				(hide yes)
+			)
+		)
 		(pin "1"
 		)
@@
 		)
 		(property "Description" "2508051027Y1"
+			(at 134.62 160.02 0)
+			(effects
+				(font
+					(size 1.27 1.27)
+				)
+				(hide yes)
+			)
+		)
+		(property "LCSC" "C85835"
 			(at 134.62 160.02 0)
 			(effects
@@
 			)
 		)
+		(property "LCSC" "C840103"
+			(at 99.06 172.72 0)
+			(effects
+				(font
+					(size 1.27 1.27)
+				)
+				(hide yes)
+			)
+		)
 		(pin "3"
 		)
@@
 			)
 		)
+		(property "LCSC" "C25905"
+			(at 208.28 71.12 0)
+			(effects
+				(font
+					(size 1.27 1.27)
+				)
+				(hide yes)
+			)
+		)
 		(pin "2"
 		)
@@
 			)
 		)
+		(property "LCSC" "C221666"
+			(at 215.9 130.81 0)
+			(effects
+				(font
+					(size 1.27 1.27)
+				)
+				(hide yes)
+			)
+		)
 		(pin "3"
 		)
@@
 				(hide yes)
 			)
+		)
+		(property "LCSC" "C139797"
+			(at 99.06 114.3 0)
+			(effects
+				(font
+					(size 1.27 1.27)
+				)
+				(hide yes)
+			)

Commit message: hw: J2/J5 -> SJ-3524-SMT-TR (C20182907, in stock); routing to follow
SJ-3523-SMT-TR (C4991872) has no JLC stock.  The SJ-3524 is the same
Same Sky SJ-352X-SMT body with a tip-switch terminal, pin 4, behind the
jack: footprint BreakoutLibrary:SJ3524SMTTR, pad 4 left unconnected.

Not routed yet.  Pad 4 sits on J6 pad 1 and the +3.3V/GND tracks and via
behind J2, and on R3/R4/FB2 and their tracks and via behind J5: 43 new DRC
items, all on pad 4.

Co-Authored-By: Claude Opus 5.5 <noreply@anthropic.com>
Claude-Session: https://claude.ai/code/session_0133r6nzUahChJ5bbJy715cX
Parts:
- J2, J5: value SJ-3523-SMT-TR -> SJ-3524-SMT-TR; footprint BreakoutLibrary:SJ3523SMTTR -> BreakoutLibrary:SJ3524SMTTR; LCSC C4991872 -> C20182907; Manufacturer_Part_Number SJ-3523-SMT-TR -> SJ-3524-SMT-TR; Mouser Part Number 490-SJ-3523-SMT-TR -> 490-SJ-3524-SMT-TR; Mouser Price/Stock https://www.mouser.co.uk/ProductDetail/CUI-Devices/SJ-3523-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 -> https://www.mouser.com/ProductDetail/Same-Sky/SJ-3524-SMT-TR
Changed lines of the file:
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@@
 			)
 		)
-		(property "Value" "SJ-3523-SMT-TR"
+		(property "Value" "SJ-3524-SMT-TR"
 			(at 88.9 63.5 0)
 			(effects
@@
 			)
 		)
-		(property "Footprint" "BreakoutLibrary:SJ3523SMTTR"
+		(property "Footprint" "BreakoutLibrary:SJ3524SMTTR"
 			(at 100.33 163.5 0)
 			(effects
@@
 			)
 		)
-		(property "Datasheet" "https://www.sameskydevices.com/product/resource/SJ-3523-SMT-TR.pdf"
+		(property "Datasheet" "https://www.sameskydevices.com/product/resource/sj-352x-smt.pdf"
 			(at 100.33 263.5 0)
 			(effects
@@
 			)
 		)
-		(property "Description" "SJ-3523-SMT-TR - 3.5 mm, Stereo, Right Angle, Surface Mount (SMT), 3 Conductors, 0 Internal Switches, Audio Jack Connector"
+		(property "Description" "SJ-3524-SMT-TR - 3.5 mm, Stereo, Right Angle, Surface Mount (SMT), 3 Conductors, 1 Internal Switch (tip), Audio Jack Connector"
 			(at 73.66 68.58 0)
 			(effects
@@
 			)
 		)
-		(property "Mouser Part Number" "490-SJ-3523-SMT-TR"
+		(property "Mouser Part Number" "490-SJ-3524-SMT-TR"
 			(at 100.33 563.5 0)
 			(effects
@@
 			)
 		)
-		(property "Mouser Price/Stock" "https://www.mouser.co.uk/ProductDetail/CUI-Devices/SJ-3523-SMT-TR?qs=WyjlAZoYn51zOHzJ3r4ZRA%3D%3D"
+		(property "Mouser Price/Stock" "https://www.mouser.com/ProductDetail/Same-Sky/SJ-3524-SMT-TR"
 			(at 100.33 663.5 0)
 			(effects
@@
 			)
 		)
-		(property "Manufacturer_Part_Number" "SJ-3523-SMT-TR"
+		(property "Manufacturer_Part_Number" "SJ-3524-SMT-TR"
 			(at 100.33 863.5 0)
 			(effects
@@
 			)
 		)
-		(property "LCSC" "C4991872"
+		(property "LCSC" "C20182907"
 			(at 73.66 68.58 0)
 			(effects
@@
 			)
 		)
-		(property "Value" "SJ-3523-SMT-TR"
+		(property "Value" "SJ-3524-SMT-TR"
 			(at 232.41 149.86 0)
 			(effects
@@
 			)
 		)
-		(property "Footprint" "BreakoutLibrary:SJ3523SMTTR"
+		(property "Footprint" "BreakoutLibrary:SJ3524SMTTR"
 			(at 243.84 249.86 0)
 			(effects
@@
 			)
 		)
-		(property "Datasheet" "https://www.sameskydevices.com/product/resource/SJ-3523-SMT-TR.pdf"
+		(property "Datasheet" "https://www.sameskydevices.com/product/resource/sj-352x-smt.pdf"
 			(at 243.84 349.86 0)
 			(effects
@@
 			)
 		)
-		(property "Description" "SJ-3523-SMT-TR - 3.5 mm, Stereo, Right Angle, Surface Mount (SMT), 3 Conductors, 0 Internal Switches, Audio Jack Connector"
+		(property "Description" "SJ-3524-SMT-TR - 3.5 mm, Stereo, Right Angle, Surface Mount (SMT), 3 Conductors, 1 Internal Switch (tip), Audio Jack Connector"
 			(at 217.17 154.94 0)
 			(effects
@@
 			)
 		)
-		(property "Mouser Part Number" "490-SJ-3523-SMT-TR"
+		(property "Mouser Part Number" "490-SJ-3524-SMT-TR"
 			(at 243.84 649.86 0)
 			(effects
@@
 			)
 		)
-		(property "Mouser Price/Stock" "https://www.mouser.co.uk/ProductDetail/CUI-Devices/SJ-3523-SMT-TR?qs=WyjlAZoYn51zOHzJ3r4ZRA%3D%3D"
+		(property "Mouser Price/Stock" "https://www.mouser.com/ProductDetail/Same-Sky/SJ-3524-SMT-TR"
 			(at 243.84 749.86 0)
 			(effects
@@
 			)
 		)
-		(property "Manufacturer_Part_Number" "SJ-3523-SMT-TR"
+		(property "Manufacturer_Part_Number" "SJ-3524-SMT-TR"
 			(at 243.84 949.86 0)
 			(effects
@@
 			)
 		)
-		(property "LCSC" "C4991872"
+		(property "LCSC" "C20182907"
 			(at 217.17 154.94 0)
 			(effects

Commit message: hw: J2/J5 -> XKB PJ-320B-SMT (C2884998), schematic + library; layout to follow
No pin behind the jack: three contacts, no switch, all copper inside the
body length.  Rated 500 mA (the SOFNG PJ-320B, C22355831, is rated 25 mA).

- BreakoutLibrary symbol PJ-320B-SMT: the SJ-3523 symbol, same pin
  positions so the wiring is untouched, renumbered to XKB's pins:
  3 sleeve, 2 ring, 4 tip (XKB X-PJ-320B-SMT rev A1; pins match SOFNG's
  A/B/C and the plug's sleeve/ring/tip order front to back)
- BreakoutLibrary.pretty/PJ-320B-SMT: pads 1.5 x 3.0 at (-3,+4) 3,
  (-1,-4) 2, (+4,+4) 4; NPTH 1.2 at (+-3, 0); origin = peg midpoint;
  plug enters from -X
- BreakoutLibrary.3dshapes/PJ-320B-SMT.step (+ .py): built from the
  drawing, none published
- project.db: J2/J5 = PJ-320B-SMT, C2884998

Board not updated: Update PCB from Schematic swaps the footprints.

Co-Authored-By: Claude Opus 5.5 <noreply@anthropic.com>
Claude-Session: https://claude.ai/code/session_0133r6nzUahChJ5bbJy715cX
Parts:
- J2, J5: value SJ-3524-SMT-TR -> PJ-320B-SMT; footprint BreakoutLibrary:SJ3524SMTTR -> BreakoutLibrary:PJ-320B-SMT; symbol DongleLibrary:SJ-3523-SMT-TR -> BreakoutLibrary:PJ-320B-SMT; Height 5.2 -> 5; LCSC C20182907 -> C2884998; Manufacturer_Name Same Sky -> XKB Connection; Manufacturer_Part_Number SJ-3524-SMT-TR -> PJ-320B-SMT; Mouser Part Number 490-SJ-3524-SMT-TR -> (none); Mouser Price/Stock https://www.mouser.com/ProductDetail/Same-Sky/SJ-3524-SMT-TR -> (none)
Connections:
- net GND: now also J2.3 (SLEEVE), J5.3 (SLEEVE); no longer J2.1 (SLEEVE), J5.1 (SLEEVE)
- net HP_L: now also J2.2 (RING); no longer J2.3 (RING)
- net HP_R: now also J2.4 (TIP); no longer J2.2 (TIP)
- net J5_RING: now also J5.2 (RING); no longer J5.3 (RING)
- net J5_TIP: now also J5.4 (TIP); no longer J5.2 (TIP)
Changed lines of the file:
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@@
 	)
 	(symbol
-		(lib_id "DongleLibrary:SJ-3523-SMT-TR")
+		(lib_id "BreakoutLibrary:PJ-320B-SMT")
 		(at 73.66 68.58 0)
 		(unit 1)
@@
 			)
 		)
-		(property "Value" "SJ-3524-SMT-TR"
+		(property "Value" "PJ-320B-SMT"
 			(at 88.9 63.5 0)
 			(effects
@@
 			)
 		)
-		(property "Footprint" "BreakoutLibrary:SJ3524SMTTR"
+		(property "Footprint" "BreakoutLibrary:PJ-320B-SMT"
 			(at 100.33 163.5 0)
 			(effects
@@
 			)
 		)
-		(property "Datasheet" "https://www.sameskydevices.com/product/resource/sj-352x-smt.pdf"
+		(property "Datasheet" "https://www.lcsc.com/product-detail/C2884998.html"
 			(at 100.33 263.5 0)
 			(effects
@@
 			)
 		)
-		(property "Description" "SJ-3524-SMT-TR - 3.5 mm, Stereo, Right Angle, Surface Mount (SMT), 3 Conductors, 1 Internal Switch (tip), Audio Jack Connector"
+		(property "Description" "PJ-320B-SMT - 3.5 mm stereo jack, right angle, SMT, 3 conductors, no switch (XKB, LCSC C2884998). Pins: 3 sleeve, 2 ring, 4 tip"
 			(at 73.66 68.58 0)
 			(effects
@@
 			)
 		)
-		(property "Height" "5.2"
+		(property "Height" "5"
 			(at 100.33 463.5 0)
 			(effects
@@
 			)
 		)
-		(property "Mouser Part Number" "490-SJ-3524-SMT-TR"
-			(at 100.33 563.5 0)
-			(effects
-				(font
-					(size 1.27 1.27)
-				)
-				(justify left top)
-				(hide yes)
-			)
-		)
-		(property "Mouser Price/Stock" "https://www.mouser.com/ProductDetail/Same-Sky/SJ-3524-SMT-TR"
-			(at 100.33 663.5 0)
-			(effects
-				(font
-					(size 1.27 1.27)
-				)
-				(justify left top)
-				(hide yes)
-			)
-		)
-		(property "Manufacturer_Name" "Same Sky"
+		(property "Manufacturer_Name" "XKB Connection"
 			(at 100.33 763.5 0)
 			(effects
@@
 			)
 		)
-		(property "Manufacturer_Part_Number" "SJ-3524-SMT-TR"
+		(property "Manufacturer_Part_Number" "PJ-320B-SMT"
 			(at 100.33 863.5 0)
 			(effects
@@
 			)
 		)
-		(property "LCSC" "C20182907"
+		(property "LCSC" "C2884998"
 			(at 73.66 68.58 0)
 			(effects
@@
 			)
 		)
-		(pin "1"
+		(pin "3"
+		)
+		(pin "4"
 		)
 		(pin "2"
-		)
-		(pin "3"
 		)
 		(instances
@@
 	)
 	(symbol
-		(lib_id "DongleLibrary:SJ-3523-SMT-TR")
+		(lib_id "BreakoutLibrary:PJ-320B-SMT")
 		(at 217.17 154.94 0)
 		(unit 1)
@@
 			)
 		)
-		(property "Value" "SJ-3524-SMT-TR"
+		(property "Value" "PJ-320B-SMT"
 			(at 232.41 149.86 0)
 			(effects
@@
 			)
 		)
-		(property "Footprint" "BreakoutLibrary:SJ3524SMTTR"
+		(property "Footprint" "BreakoutLibrary:PJ-320B-SMT"
 			(at 243.84 249.86 0)
 			(effects
@@
 			)
 		)
-		(property "Datasheet" "https://www.sameskydevices.com/product/resource/sj-352x-smt.pdf"
+		(property "Datasheet" "https://www.lcsc.com/product-detail/C2884998.html"
 			(at 243.84 349.86 0)
 			(effects
@@
 			)
 		)
-		(property "Description" "SJ-3524-SMT-TR - 3.5 mm, Stereo, Right Angle, Surface Mount (SMT), 3 Conductors, 1 Internal Switch (tip), Audio Jack Connector"
+		(property "Description" "PJ-320B-SMT - 3.5 mm stereo jack, right angle, SMT, 3 conductors, no switch (XKB, LCSC C2884998). Pins: 3 sleeve, 2 ring, 4 tip"
 			(at 217.17 154.94 0)
 			(effects
@@
 			)
 		)
-		(property "Height" "5.2"
+		(property "Height" "5"
 			(at 243.84 549.86 0)
 			(effects
@@
 			)
 		)
-		(property "Mouser Part Number" "490-SJ-3524-SMT-TR"
-			(at 243.84 649.86 0)
-			(effects
-				(font
-					(size 1.27 1.27)
-				)
-				(justify left top)
-				(hide yes)
-			)
-		)
-		(property "Mouser Price/Stock" "https://www.mouser.com/ProductDetail/Same-Sky/SJ-3524-SMT-TR"
-			(at 243.84 749.86 0)
-			(effects
-				(font
-					(size 1.27 1.27)
-				)
-				(justify left top)
-				(hide yes)
-			)
-		)
-		(property "Manufacturer_Name" "Same Sky"
+		(property "Manufacturer_Name" "XKB Connection"
 			(at 243.84 849.86 0)
 			(effects
@@
 			)
 		)
-		(property "Manufacturer_Part_Number" "SJ-3524-SMT-TR"
+		(property "Manufacturer_Part_Number" "PJ-320B-SMT"
 			(at 243.84 949.86 0)
 			(effects
@@
 			)
 		)
-		(property "LCSC" "C20182907"
+		(property "LCSC" "C2884998"
 			(at 217.17 154.94 0)
 			(effects
@@
 			)
 		)
-		(pin "1"
+		(pin "3"
+		)
+		(pin "4"
 		)
 		(pin "2"
 		)
-		(pin "3"
-		)
 		(instances
